File: HW/H3S-Dev-V1/H3S-Dev-V1.kicad_pcb (KiCad board)
At the start: 2 copper layers, 85 x 56 mm, 38 parts, among them J1 USB_C_Receptacle_USB2.0_16P, J2 Conn_01x02_Socket, J3 Conn_Coaxial, Q1 DMP3099L, SW1 SW_Push, U1 Ai-Thinker-Ra-01, U2 LTC4054ES5-4.2, U3 USBLC6-2SC6, U4 ESP32-S3-WROOM-1, U5 SY8089AAAC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

Commit message: Some progress...
Parts:
- added J4: Conn_01x04, Connector:NS-Tech_Grove_1x04_P2mm_Vertical, F.Cu at (161.5, 84.0)
- added J5: Conn_01x04, Connector:NS-Tech_Grove_1x04_P2mm_Vertical, F.Cu at (171.5, 84.0)
- added R12: 10k, Resistor_SMD:R_0603_1608Metric, F.Cu at (155.9, 84.0)
- added R13: 10k, Resistor_SMD:R_0603_1608Metric, F.Cu at (155.9, 86.0)
- added R14: 10k, Resistor_SMD:R_0603_1608Metric, F.Cu at (176.2, 84.0)
- added R15: 10k, Resistor_SMD:R_0603_1608Metric, F.Cu at (176.2, 86.0)
- added R16: 0, Resistor_SMD:R_0603_1608Metric, F.Cu at (171.7, 110.6)
- moved H2 20.0 mm to (161.5, 77.5)
- moved H4 20.0 mm to (161.5, 126.5)
- moved SW1 8.98 mm to (127.2, 104.8)
- moved U4 8.31 mm to (142.6, 102.0)
- moved C4 4.69 mm to (146.5, 118.0)
- moved C5 4.69 mm to (146.5, 115.8)
- moved C6 4.69 mm to (144.2, 123.8)
- moved C7 4.69 mm to (150.3, 119.7)
- moved L1 4.69 mm to (152.6, 123.2)
- moved Q1 4.69 mm to (140.9, 116.7)
- moved R10 4.69 mm to (144.1, 127.0)
- moved R9 4.69 mm to (144.1, 125.5)
- moved U5 4.69 mm to (148.0, 122.8)
- moved C3 4.69 mm to (146.3, 119.8)
- moved D3 4.69 mm to (141.6, 119.8)
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Connections:
- U4 pad 38: unconnected-(U4-IO2-Pad38) -> /SCL
- U4 pad 39: unconnected-(U4-IO1-Pad39) -> /SDA
- U6 pad 1: (no net) -> Net-(U6-VCC_IO)
- U6 pad 10: unconnected-(U6-GND__2-Pad10) -> GND
- U6 pad 11: unconnected-(U6-GND__3-Pad11) -> GND
- U6 pad 12: unconnected-(U6-GND__4-Pad12) -> GND
- U6 pad 13: unconnected-(U6-GND__5-Pad13) -> GND
- U6 pad 14: unconnected-(U6-GND__6-Pad14) -> GND
- U6 pad 15: unconnected-(U6-GND__7-Pad15) -> GND
- U6 pad 16: unconnected-(U6-RF_OUT-Pad16) -> Net-(U6-RF_IN)
- U6 pad 17: unconnected-(U6-RF_IN-Pad17) -> Net-(U6-RF_IN)
- U6 pad 18: unconnected-(U6-GND__8-Pad18) -> GND
- U6 pad 19: unconnected-(U6-GND__9-Pad19) -> GND
- U6 pad 21: unconnected-(U6-GND__10-Pad21) -> GND
- U6 pad 22: unconnected-(U6-GND__11-Pad22) -> GND
- U6 pad 27: unconnected-(U6-GND__12-Pad27) -> GND
- U6 pad 30: unconnected-(U6-ANTON-Pad30) -> GND
- U6 pad 31: unconnected-(U6-GND__13-Pad31) -> GND
- U6 pad 4: unconnected-(U6-GND-Pad4) -> GND
- U6 pad 5: unconnected-(U6-GND__1-Pad5) -> GND
- U6 pad 8: unconnected-(U6-V_BCKP-Pad8) -> VCC
- U6 pad 9: unconnected-(U6-VCC-Pad9) -> VCC
Routing:
- net /~{LoRa_RST}: track 44.7 -> 0.00 mm, vias 1 -> 0
- net /DIO0: track 39.2 -> 0.00 mm, vias 1 -> 0
- net /DIO2: track 37.9 -> 0.00 mm, vias 1 -> 0
- net /DIO1: track 36.0 -> 0.00 mm, vias 1 -> 0
- net /MISO: track 34.1 -> 0.00 mm, vias 1 -> 0
- net /~{SS}: track 32.1 -> 0.00 mm, vias 1 -> 0
- net /MOSI: track 21.6 -> 0.00 mm, vias 1 -> 0
- net VCC: track 36.8 -> 19.1 mm, vias 5 -> 3
- net /SCK: track 15.8 -> 0.00 mm, vias 1 -> 0
- net /~{ESP_EN}: track 12.8 -> 4.34 mm
- net /VBUS: track 59.7 -> 55.0 mm
- net /VBAT: track 29.4 -> 26.5 mm
- net Net-(U6-RF_IN): track 0.00 -> 1.00 mm
- net /V5_SENSE: track 7.97 -> 7.18 mm

Commit message: RA-01SH-P LoRa module added
Parts:
- U1: value Ai-Thinker-Ra-01 -> Ra-01SH-P; footprint RF_Module:Ai-Thinker-Ra-01-LoRa -> H3S-Dev:Ra-01SH-P
Connections:
- net /~{LoRa_RST} renamed /~{L_RST}
- U1 pad 10: /DIO4 -> unconnected-(U1-BUSY-Pad10)
- U1 pad 11: /DIO5 -> unconnected-(U1-RF_EN-Pad11)
- U1 pad 5: /DIO0 -> unconnected-(U1-VCCPA-Pad5)
- U1 pad 6: /DIO1 -> /DIO0
- U1 pad 7: /DIO2 -> /DIO1
- U1 pad 8: /DIO3 -> /DIO2

Commit message: J2 updated
Parts:
- J2: value Conn_01x02_Socket -> Conn_01x02
- moved J2 0.10 mm to (124.4, 125.2)

Commit message: LoRa updates
Parts:
- added C10: NA, Capacitor_SMD:C_0603_1608Metric, F.Cu at (110.3, 86.3)
- added C11: NA, Capacitor_SMD:C_0603_1608Metric, F.Cu at (108.7, 86.3)
- added R17: 0, Resistor_SMD:R_0603_1608Metric, F.Cu at (128.3, 111.2)
- added R18: 0, Resistor_SMD:R_0603_1608Metric, F.Cu at (109.5, 83.6)
- added R19: 0, Resistor_SMD:R_0603_1608Metric, F.Cu at (108.8, 91.7)
- moved U1 5.57 mm to (121.8, 90.7)
- moved R11 5.20 mm to (136.1, 95.4)
- moved C8 5.20 mm to (134.2, 95.5)
- moved C9 5.20 mm to (132.4, 95.4)
- moved U4 5.20 mm to (147.8, 102.1)
- moved SW1 5.15 mm to (132.3, 105.0)
- moved J3 2.21 mm to (106.0, 83.6)
Connections:
- U1 pad 1: Net-(J3-In) -> Net-(U1-ANT)
- U1 pad 10: unconnected-(U1-BUSY-Pad10) -> /L_BUSY
- U1 pad 11: unconnected-(U1-RF_EN-Pad11) -> Net-(U1-RF_EN)
- U1 pad 5: unconnected-(U1-VCCPA-Pad5) -> Net-(U1-VCCPA)
- U4 pad 21: unconnected-(U4-IO13-Pad21) -> /L_BUSY
- U4 pad 22: unconnected-(U4-IO14-Pad22) -> /L_RF_EN
- U4 pad 31: unconnected-(U4-IO38-Pad31) -> /BAT_SENSE
- U4 pad 32: unconnected-(U4-IO39-Pad32) -> /V5_SENSE

Commit message: Minor changes
Parts:
- C10, C11: footprint Capacitor_SMD:C_0603_1608Metric -> Capacitor_SMD:C_0402_1005Metric
- R18: footprint Resistor_SMD:R_0603_1608Metric -> Resistor_SMD:R_0402_1005Metric
- moved C10 2.62 mm to (111.8, 84.2)
- moved C11 2.16 mm to (108.8, 84.2)
- moved R18 0.75 mm to (110.2, 83.7)
- moved J3 0.11 mm to (106.1, 83.7)
Routing:
- net Net-(U1-ANT): track 0.00 -> 3.06 mm
- net Net-(J3-In): track 0.00 -> 2.61 mm
Changed lines of the file:
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@@
 	(footprint "Connector_Coaxial:U.FL_Hirose_U.FL-R-SMT-1_Vertical"
 		(layer "F.Cu")
-		(at 106 83.61 180)
+		(at 106.1 83.65 180)
 		(descr "Hirose U.FL Coaxial https://www.hirose.com/product/en/products/U.FL/U.FL-R-SMT-1%2810%29/")
 		(tags "Hirose U.FL Coaxial")
@@
 			(polygon
 				(pts
-					(xy 104.425 84.56) (xy 106.515 84.56) (xy 106.515 82.66) (xy 104.425 82.66)
+					(xy 104.525 84.6) (xy 106.615 84.6) (xy 106.615 82.7) (xy 104.525 82.7)
 				)
 			)
@@
 		)
 	)
-	(footprint "Capacitor_SMD:C_0603_1608Metric"
+	(footprint "Capacitor_SMD:C_0402_1005Metric"
 		(layer "F.Cu")
-		(at 110.3 86.26 -90)
-		(descr "Capacitor SMD 0603 (1608 Metric), square (rectangular) end terminal, IPC-7351 nominal, (Body size source: IPC-SM-782 page 76, https://www.pcb-3d.com/wordpress/wp-content/uploads/ipc-sm-782a_amendment_1_and_2.pdf), generated with kicad-footprint-generator")
+		(at 111.85 84.15 -90)
+		(descr "Capacitor SMD 0402 (1005 Metric), square (rectangular) end terminal, IPC-7351 nominal, (Body size source: IPC-SM-782 page 76, https://www.pcb-3d.com/wordpress/wp-content/uploads/ipc-sm-782a_amendment_1_and_2.pdf), generated with kicad-footprint-generator")
 		(tags "capacitor")
 		(property "Reference" "C10"
-			(at 0 -1.43 90)
+			(at 2.3 0.75 270)
 			(layer "F.SilkS")
 			(effects
@@
 		)
 		(property "Value" "NA"
-			(at 0 1.43 90)
+			(at 0 1.16 270)
 			(layer "F.Fab")
 			(hide yes)
@@
 		)
 		(property "Datasheet" "~"
-			(at 0 0 90)
+			(at 0 0 270)
 			(layer "F.Fab")
 			(hide yes)
@@
 		)
 		(property "Description" "Unpolarized capacitor"
-			(at 0 0 90)
+			(at 0 0 270)
 			(layer "F.Fab")
 			(hide yes)
@@
 		(attr smd)
 		(fp_line
-			(start -0.14058 0.51)
-			(end 0.14058 0.51)
+			(start -0.107836 0.36)
+			(end 0.107836 0.36)
 			(stroke
 				(width 0.12)
@@
 		)
 		(fp_line
-			(start -0.14058 -0.51)
-			(end 0.14058 -0.51)
+			(start -0.107836 -0.36)
+			(end 0.107836 -0.36)
 			(stroke
 				(width 0.12)
@@
 		)
 		(fp_rect
-			(start -1.48 -0.73)
-			(end 1.48 0.73)
+			(start -0.91 -0.46)
+			(end 0.91 0.46)
 			(stroke
 				(width 0.05)
@@
 		)
 		(fp_rect
-			(start -0.8 -0.4)
-			(end 0.8 0.4)
+			(start -0.5 -0.25)
+			(end 0.5 0.25)
 			(stroke
 				(width 0.1)
@@
 		)
 		(fp_text user "${REFERENCE}"
-			(at 0 0 90)
+			(at 0 0 270)
 			(layer "F.Fab")
 			(effects
 				(font
-					(size 0.4 0.4)
-					(thickness 0.06)
+					(size 0.25 0.25)
+					(thickness 0.04)
 				)
 			)
 		)
 		(pad "1" smd roundrect
-			(at -0.775 0 270)
-			(size 0.9 0.95)
+			(at -0.48 0 270)
+			(size 0.56 0.62)
 			(layers "F.Cu" "F.Mask" "F.Paste")
 			(roundrect_rratio 0.25)
@@
 		)
 		(pad "2" smd roundrect
-			(at 0.775 0 270)
-			(size 0.9 0.95)
+			(at 0.48 0 270)
+			(size 0.56 0.62)
 			(layers "F.Cu" "F.Mask" "F.Paste")
 			(roundrect_rratio 0.25)
@@
 		)
 		(embedded_fonts no)
-		(model "${KICAD9_3DMODEL_DIR}/Capacitor_SMD.3dshapes/C_0603_1608Metric.step"
+		(model "${KICAD9_3DMODEL_DIR}/Capacitor_SMD.3dshapes/C_0402_1005Metric.step"
 			(offset
 				(xyz 0 0 0)
@@
 		)
 	)
-	(footprint "Capacitor_SMD:C_0603_1608Metric"
+	(footprint "Capacitor_SMD:C_0402_1005Metric"
 		(layer "F.Cu")
-		(at 108.65 86.31 -90)
-		(descr "Capacitor SMD 0603 (1608 Metric), square (rectangular) end terminal, IPC-7351 nominal, (Body size source: IPC-SM-782 page 76, https://www.pcb-3d.com/wordpress/wp-content/uploads/ipc-sm-782a_amendment_1_and_2.pdf), generated with kicad-footprint-generator")
+		(at 108.75 84.15 -90)
+		(descr "Capacitor SMD 0402 (1005 Metric), square (rectangular) end terminal, IPC-7351 nominal, (Body size source: IPC-SM-782 page 76, https://www.pcb-3d.com/wordpress/wp-content/uploads/ipc-sm-782a_amendment_1_and_2.pdf), generated with kicad-footprint-generator")
 		(tags "capacitor")
 		(property "Reference" "C11"
-			(at -2.8 0 90)
+			(at 2.24 0 270)
 			(layer "F.SilkS")
 			(effects
@@
 		)
 		(property "Value" "NA"
-			(at 0 1.43 90)
+			(at 0 1.16 270)
 			(layer "F.Fab")
 			(hide yes)
@@
 		)
 		(property "Datasheet" "~"
-			(at 0 0 90)
+			(at 0 0 270)
 			(layer "F.Fab")
 			(hide yes)
@@
 		)
 		(property "Description" "Unpolarized capacitor"
-			(at 0 0 90)
+			(at 0 0 270)
 			(layer "F.Fab")
 			(hide yes)
@@
 		(attr smd)
 		(fp_line
-			(start -0.14058 0.51)
-			(end 0.14058 0.51)
+			(start -0.107836 0.36)
+			(end 0.107836 0.36)
 			(stroke
 				(width 0.12)
@@
 		)
 		(fp_line
-			(start -0.14058 -0.51)
-			(end 0.14058 -0.51)
+			(start -0.107836 -0.36)
+			(end 0.107836 -0.36)
 			(stroke
 				(width 0.12)
@@
 		)
 		(fp_rect
-			(start -1.48 -0.73)
-			(end 1.48 0.73)
+			(start -0.91 -0.46)
+			(end 0.91 0.46)
 			(stroke
 				(width 0.05)
@@
 		)
 		(fp_rect
-			(start -0.8 -0.4)
-			(end 0.8 0.4)
+			(start -0.5 -0.25)
+			(end 0.5 0.25)
 			(stroke
 				(width 0.1)
@@
 		)
 		(fp_text user "${REFERENCE}"
-			(at 0 0 90)
+			(at 0 0 270)
 			(layer "F.Fab")
 			(effects
 				(font
-					(size 0.4 0.4)
-					(thickness 0.06)
+					(size 0.25 0.25)
+					(thickness 0.04)
 				)
 			)
 		)
 		(pad "1" smd roundrect
-			(at -0.775 0 270)
-			(size 0.9 0.95)
+			(at -0.48 0 270)
+			(size 0.56 0.62)
 			(layers "F.Cu" "F.Mask" "F.Paste")
 			(roundrect_rratio 0.25)
@@
 		)
 		(pad "2" smd roundrect
-			(at 0.775 0 270)
-			(size 0.9 0.95)
+			(at 0.48 0 270)
+			(size 0.56 0.62)
 			(layers "F.Cu" "F.Mask" "F.Paste")
 			(roundrect_rratio 0.25)
@@
 		)
 		(embedded_fonts no)
-		(model "${KICAD9_3DMODEL_DIR}/Capacitor_SMD.3dshapes/C_0603_1608Metric.step"
+		(model "${KICAD9_3DMODEL_DIR}/Capacitor_SMD.3dshapes/C_0402_1005Metric.step"
 			(offset
 				(xyz 0 0 0)
@@
 		)
 	)
-	(footprint "Resistor_SMD:R_0603_1608Metric"
+	(footprint "Resistor_SMD:R_0402_1005Metric"
 		(layer "F.Cu")
-		(at 109.5 83.61 180)
-		(descr "Resistor SMD 0603 (1608 Metric), square (rectangular) end terminal, IPC-7351 nominal, (Body size source: IPC-SM-782 page 72, https://www.pcb-3d.com/wordpress/wp-content/uploads/ipc-sm-782a_amendment_1_and_2.pdf), generated with kicad-footprint-generator")
+		(at 110.25 83.65 180)
+		(descr "Resistor SMD 0402 (1005 Metric), square (rectangular) end terminal, IPC-7351 nominal, (Body size source: IPC-SM-782 page 72, https://www.pcb-3d.com/wordpress/wp-content/uploads/ipc-sm-782a_amendment_1_and_2.pdf), generated with kicad-footprint-generator")
 		(tags "resistor")
 		(property "Reference" "R18"
-			(at 0 -1.43 0)
+			(at 0 1.3 180)
 			(layer "F.SilkS")
 			(effects
@@
 		)
 		(property "Value" "0"
-			(at 0 1.43 0)
+			(at 0 1.17 180)
 			(layer "F.Fab")
 			(hide yes)
@@
 		)
 		(property "Datasheet" "~"
-			(at 0 0 0)
+			(at 0 0 180)
 			(layer "F.Fab")
 			(hide yes)
@@
 		)
 		(property "Description" "Resistor"
-			(at 0 0 0)
+			(at 0 0 180)
 			(layer "F.Fab")
 			(hide yes)
@@
 		(attr smd)
 		(fp_line
-			(start -0.237258 0.5225)
-			(end 0.237258 0.5225)
+			(start -0.153641 0.38)
+			(end 0.153641 0.38)
 			(stroke
 				(width 0.12)
@@
 		)
 		(fp_line
-			(start -0.237258 -0.5225)
-			(end 0.237258 -0.5225)
+			(start -0.153641 -0.38)
+			(end 0.153641 -0.38)
 			(stroke
 				(width 0.12)
@@
 		)
 		(fp_rect
-			(start -1.48 -0.73)
-			(end 1.48 0.73)
+			(start -0.93 -0.47)
+			(end 0.93 0.47)
 			(stroke
 				(width 0.05)
@@
 		)
 		(fp_rect
-			(start -0.8 -0.4125)
-			(end 0.8 0.4125)
+			(start -0.525 -0.27)
+			(end 0.525 0.27)
 			(stroke
 				(width 0.1)
@@
 		)
 		(fp_text user "${REFERENCE}"
-			(at 0 0 0)
+			(at 0 0 180)
 			(layer "F.Fab")
 			(effects
 				(font
-					(size 0.4 0.4)
-					(thickness 0.06)
+					(size 0.26 0.26)
+					(thickness 0.04)
 				)
 			)
 		)
 		(pad "1" smd roundrect
-			(at -0.825 0 180)
-			(size 0.8 0.95)
+			(at -0.51 0 180)
+			(size 0.54 0.64)
 			(layers "F.Cu" "F.Mask" "F.Paste")
 			(roundrect_rratio 0.25)
@@
 		)
 		(pad "2" smd roundrect
-			(at 0.825 0 180)
-			(size 0.8 0.95)
+			(at 0.51 0 180)
+			(size 0.54 0.64)
 			(layers "F.Cu" "F.Mask" "F.Paste")
 			(roundrect_rratio 0.25)
@@
 		)
 		(embedded_fonts no)
-		(model "${KICAD9_3DMODEL_DIR}/Resistor_SMD.3dshapes/R_0603_1608Metric.step"
+		(model "${KICAD9_3DMODEL_DIR}/Resistor_SMD.3dshapes/R_0402_1005Metric.step"
 			(offset
 				(xyz 0 0 0)
@@
 	)
 	(segment
+		(start 110.78 83.67)
+		(end 110.76 83.65)
+		(width 0.2)
+		(layer "F.Cu")
+		(net 17)
+	)
+	(segment
+		(start 111.87 83.65)
+		(end 111.85 83.67)
+		(width 0.2)
+		(layer "F.Cu")
+		(net 17)
+	)
+	(segment
+		(start 113.8 83.65)
+		(end 111.87 83.65)
+		(width 0.2)
+		(layer "F.Cu")
+		(net 17)
+	)
+	(segment
+		(start 111.85 83.67)
+		(end 110.78 83.67)
+		(width 0.2)
+		(layer "F.Cu")
+		(net 17)
+	)
+	(segment
 		(start 121.8 117.85)
 		(end 121.8 119.6)
@@
 	)
 	(segment
+		(start 108.75 83.67)
+		(end 107.17 83.67)
+		(width 0.2)
+		(layer "F.Cu")
+		(net 51)
+	)
+	(segment
+		(start 109.74 83.65)
+		(end 108.77 83.65)
+		(width 0.2)
+		(layer "F.Cu")
+		(net 51)
+	)
+	(segment
+		(start 107.17 83.67)
+		(end 107.15 83.65)
+		(width 0.2)
+		(layer "F.Cu")
+		(net 51)
+	)
+	(segment
+		(start 108.77 83.65)
+		(end 108.75 83.67)
+		(width 0.2)
+		(layer "F.Cu")
+		(net 51)
+	)
+	(segment

Commit message: Some progress
Parts:
- added C12: 1u, Capacitor_SMD:C_0603_1608Metric, F.Cu at (161.6, 110.9)
- added C13: 100n, Capacitor_SMD:C_0603_1608Metric, F.Cu at (159.9, 110.9)
- added D2: LED, LED_SMD:LED_0603_1608Metric, F.Cu at (166.1, 119.7)
- added D4: LED, LED_SMD:LED_0603_1608Metric, F.Cu at (164.9, 102.8)
- added R20: 10k, Resistor_SMD:R_0603_1608Metric, F.Cu at (163.2, 110.9)
- added R21: 10k, Resistor_SMD:R_0603_1608Metric, F.Cu at (164.3, 119.6)
- added R22: 10k, Resistor_SMD:R_0603_1608Metric, F.Cu at (164.9, 106.1)
- added R23: 20, Resistor_SMD:R_0603_1608Metric, F.Cu at (170.9, 94.1)
- added R24: 20, Resistor_SMD:R_0603_1608Metric, F.Cu at (172.7, 94.2)
- added R25: 20, Resistor_SMD:R_0603_1608Metric, F.Cu at (174.7, 93.9)
- added R26: 20, Resistor_SMD:R_0603_1608Metric, F.Cu at (177.6, 110.5)
- added R27: 20, Resistor_SMD:R_0603_1608Metric, F.Cu at (167.6, 101.1)
- added R28: 0, Resistor_SMD:R_0603_1608Metric, F.Cu at (176.2, 110.5)
- added R29: 0, Resistor_SMD:R_0603_1608Metric, F.Cu at (173.7, 110.5)
- added SW2: SW_Push, Button_Switch_SMD:SW_Tactile_SPST_NO_Straight_CK_PTS636Sx25SMTRLFS, F.Cu at (161.5, 98.9)
Connections:
- U4 pad 27: unconnected-(U4-IO0-Pad27) -> /~{ESP_IO0}
- U6 pad 2: unconnected-(U6-3D_FIX-Pad2) -> /G_3D
- U6 pad 20: unconnected-(U6-JAM_DET-Pad20) -> /G_JD
- U6 pad 23: unconnected-(U6-~{RESET}-Pad23) -> /~{G_RESET}
- U6 pad 24: unconnected-(U6-GEO_FENCE-Pad24) -> /G_GF
- U6 pad 25: unconnected-(U6-TXD1-Pad25) -> /G_TX
- U6 pad 26: unconnected-(U6-RXD1-Pad26) -> /G_RX
- U6 pad 28: unconnected-(U6-FORCE_ON-Pad28) -> /G_FO
- U6 pad 29: unconnected-(U6-TIMEPULSE-Pad29) -> /G_TP
- U6 pad 3: unconnected-(U6-I2C_SDA-Pad3) -> /G_SDA
- U6 pad 6: unconnected-(U6-I2C_SCL-Pad6) -> /G_SCL
- U6 pad 7: unconnected-(U6-EXTINT0-Pad7) -> /G_INT

Commit message: Some progress
Parts:
- added R30: 0, Resistor_SMD:R_0603_1608Metric, F.Cu at (165.1, 102.4)
- added R31: 0, Resistor_SMD:R_0603_1608Metric, F.Cu at (172.7, 112.6)
- added R32: 0, Resistor_SMD:R_0603_1608Metric, F.Cu at (175.4, 91.3)
- added R33: 0, Resistor_SMD:R_0603_1608Metric, F.Cu at (178.4, 91.3)
- moved R17 20.4 mm to (108.8, 105.2), turned to -90 degrees
- moved SW2 14.6 mm to (158.0, 113.0), turned to 0 degrees
- moved C8 14.1 mm to (128.1, 108.2)
- moved R11 14.1 mm to (129.9, 108.1)
- moved C9 14.1 mm to (126.3, 108.1)
- moved J3 13.9 mm to (118.8, 78.1), turned to 90 degrees
- moved R19 11.1 mm to (110.8, 80.8), turned to -90 degrees
- moved U1 10.5 mm to (111.8, 93.8), turned to -90 degrees
- moved C11 10.1 mm to (118.3, 80.8), turned to 180 degrees
- moved SW1 9.11 mm to (128.0, 113.0), turned to 180 degrees
- moved R12 9.07 mm to (164.0, 88.0), turned to 180 degrees
- moved R18 8.67 mm to (118.8, 82.3), turned to 90 degrees
- moved R15 7.82 mm to (175.7, 78.2)
- moved R20 7.49 mm to (156.4, 107.8), turned to -90 degrees
- moved J5 7.04 mm to (178.5, 84.0), turned to -90 degrees
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Other:
- board text added: "H3S-Dev-V1 by HobbyIoT"
- board text added: "Meshtastic node Helium node"
- board text removed: "(c) HobbyIoT H3S-Dev-V1 Helium node Meshtastic node"

Commit message: Some progress
Parts:
- moved R17 16.0 mm to (124.3, 101.5), turned to 0 degrees
- moved C12 2.59 mm to (159.2, 105.5)
- moved C13 2.59 mm to (160.9, 105.5)
- moved R20 2.59 mm to (157.6, 105.5)
- moved SW2 2.59 mm to (159.2, 110.7)
- moved R11 2.40 mm to (129.2, 105.8)
- moved C9 2.40 mm to (125.6, 105.8)
- moved SW1 2.40 mm to (127.3, 110.7)
- moved C8 2.40 mm to (127.4, 105.9)
- moved R19 1.44 mm to (112.2, 80.4)
- moved C10 1.44 mm to (119.7, 83.5)
- moved C11 1.44 mm to (119.7, 80.4)
- moved J3 1.44 mm to (120.2, 77.8)
- moved R18 1.44 mm to (120.2, 81.9)
- moved U1 1.44 mm to (113.2, 93.5)
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Routing:
- net (no net): vias 0 -> 83
Other:
- board text added: "Meshtastic/Helium node"
- board text removed: "Meshtastic node Helium node"
