File: HW/H3S-Dev-V1/H3S-Dev-V1.kicad_sch (KiCad schematic)
At the start: 84 parts, among them J1 USB_C_Receptacle_USB2.0_16P, J2 Conn_01x02, J3 Conn_Coaxial, J4 Conn_01x04, J5 Conn_01x04, J6 Conn_01x02, Q1 DMP3099L, SW1 SW_Push, SW2 SW_Push, U1 Ra-01SH-P, U2 LTC4054ES5-4.2, U3 USBLC6-2SC6, U4 ESP32-S3-WROOM-1, U5 SY8089AAAC, U6 L96-M33

Commit message: BOM update
Parts:
- U4: value ESP32-S3-WROOM-1 -> ESP32-S3-WROOM-1U-N16R8
Changed lines of the file:
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@@
 			)
 		)
-		(property "Description" "Resistor"
+		(property "Description" "Resistor 10k 5% 0.25W SMD 0603『 』10k"
 			(at 57.15 41.91 0)
 			(effects
@@
 			)
 		)
-		(property "Description" "Resistor"
+		(property "Description" "Resistor 10k 5% 0.25W SMD 0603『 』10k"
 			(at 269.24 220.98 0)
 			(effects
@@
 			)
 		)
-		(property "Description" "Unpolarized capacitor"
+		(property "Description" "Capacitor ceramic 100n 16V 10% X7R 0603『 』100n"
 			(at 229.87 146.05 0)
 			(effects
@@
 			)
 		)
-		(property "Description" "Unpolarized capacitor"
+		(property "Description" "Capacitor ceramic 100n 16V 10% X7R 0603『 』100n"
 			(at 107.95 219.71 0)
 			(effects
@@
 			)
 		)
-		(property "Description" "Resistor"
+		(property "Description" "Resistor 0 5% 0.25W SMD 0603『 』0 ohm"
 			(at 295.91 109.22 0)
 			(effects
@@
 			)
 		)
-		(property "Description" "Resistor"
+		(property "Description" "Resistor 0 5% 0.25W SMD 0603『 』0 ohm"
 			(at 373.38 111.76 0)
 			(effects
@@
 			)
 		)
-		(property "Description" "Resistor"
+		(property "Description" "Resistor 0 5% 0.25W SMD 0603『 』0 ohm"
 			(at 294.64 82.55 0)
 			(effects
@@
 			)
 		)
-		(property "Description" "Unpolarized capacitor"
+		(property "Description" "Capacitor ceramic 22u 6.3V 10% C0G 0805『 』22u"
 			(at 240.03 212.09 0)
 			(effects
@@
 			)
 		)
-		(property "Description" "Light emitting diode"
+		(property "Description" "LED Red SMD 0603『 』LED RED"
 			(at 123.19 189.23 0)
 			(effects
@@
 			)
 		)
-		(property "Description" "Resistor"
+		(property "Description" "Resistor 0 5% 0.25W SMD 0603『 』0 ohm"
 			(at 247.65 96.52 0)
 			(effects
@@
 			)
 		)
-		(property "Description" "Resistor"
+		(property "Description" "Resistor 22 ohm 5% 0.25W SMD 0603『 』22 ohm"
 			(at 115.57 129.54 0)
 			(effects
@@
 			)
 		)
-		(property "Description" "Unpolarized capacitor"
+		(property "Description" "Capacitor ceramic 22p 6.3V 10% C0G 0603『 』22p"
 			(at 218.44 212.09 0)
 			(effects
@@
 			)
 		)
-		(property "Description" "Unpolarized capacitor"
+		(property "Description" "Capacitor ceramic 100n 16V 10% X7R 0603『 』100n"
 			(at 271.78 146.05 0)
 			(effects
@@
 			)
 		)
-		(property "Description" "Light emitting diode"
+		(property "Description" "LED Green SMD 0603『 』LED GRN"
 			(at 208.28 151.13 0)
 			(effects
@@
 			)
 		)
-		(property "Description" "Resistor"
+		(property "Description" "Resistor 0 5% 0.25W SMD 0603『 』0 ohm"
 			(at 382.27 116.84 0)
 			(effects
@@
 			)
 		)
-		(property "Description" "Resistor"
+		(property "Description" "Resistor 10k 5% 0.25W SMD 0603『 』10k"
 			(at 48.26 73.66 0)
 			(effects
@@
 			)
 		)
-		(property "Description" "Resistor"
+		(property "Description" "Resistor 10k 5% 0.25W SMD 0603『 』10k"
 			(at 57.15 73.66 0)
 			(effects
@@
 			)
 		)
-		(property "Description" "Light emitting diode"
+		(property "Description" "LED Green SMD 0603『 』LED GRN"
 			(at 269.24 210.82 0)
 			(effects
@@
 			)
 		)
-		(property "Description" "Resistor"
+		(property "Description" "Resistor 5.1k 5% 0.25W SMD 0603『 』5.1k"
 			(at 62.23 148.59 0)
 			(effects
@@
 			)
 		)
-		(property "Description" "Unpolarized capacitor"
+		(property "Description" "Capacitor ceramic 100n 16V 10% X7R 0603『 』100n"
 			(at 83.82 219.71 0)
 			(effects
@@
 			)
 		)
-		(property "Description" "Resistor"
+		(property "Description" "Resistor 2.2k 5% 0.25W SMD 0603『 』2.2k"
 			(at 123.19 219.71 0)
 			(effects
@@
 			)
 		)
-		(property "Description" "Multi-GNSS receiver module with embedded chip antenna"
+		(property "Description" "Multi-GNSS receiver module with embedded chip antenna P/N L96-M33"
 			(at 330.2 109.22 0)
 			(effects
@@
 			)
 		)
-		(property "Description" "Resistor"
+		(property "Description" "Resistor 20 ohm 5% 0.25W SMD 0603『 』20 ohm"
 			(at 288.29 104.14 0)
 			(effects
@@
 			)
 		)
-		(property "Description" "Unpolarized capacitor"
+		(property "Description" "Capacitor ceramic 100n 16V 10% X7R 0603『 』100n"
 			(at 167.64 222.25 0)
 			(effects
@@
 			)
 		)
-		(property "Description" "Resistor"
+		(property "Description" "Resistor 49.9k 1% 0.25W SMD 0603『 』49.9k"
 			(at 231.14 215.9 0)
 			(effects
@@
 			)
 		)
-		(property "Description" "Light emitting diode"
+		(property "Description" "LED Green SMD 0603『 』LED GRN"
 			(at 367.03 151.13 0)
 			(effects
@@
 			)
 		)
-		(property "Description" "Resistor"
+		(property "Description" "Resistor 1.5k 5% 0.25W SMD 0603『 』1.5k"
 			(at 100.33 118.11 0)
 			(effects
@@
 			)
 		)
-		(property "Description" "Resistor"
+		(property "Description" "Resistor 0 5% 0.25W SMD 0603『 』0 ohm"
 			(at 199.39 78.74 0)
 			(effects
@@
 			)
 		)
-		(property "Description" "Resistor"
+		(property "Description" "Resistor 20 ohm 5% 0.25W SMD 0603『 』20 ohm"
 			(at 288.29 119.38 0)
 			(effects
@@
 			)
 		)
-		(property "Description" "Resistor"
+		(property "Description" "Resistor 0 5% 0.25W SMD 0603『 』0 ohm"
 			(at 373.38 119.38 0)
 			(effects
@@
 			)
 		)
-		(property "Description" "Resistor"
+		(property "Description" "Resistor 470k 1% 0.25W SMD 0603『 』470k"
 			(at 97.79 207.01 0)
 			(effects
@@
 			)
 		)
-		(property "Description" "Resistor"
+		(property "Description" "Resistor 20 ohm 5% 0.25W SMD 0603『 』20 ohm"
 			(at 295.91 116.84 0)
 			(effects
@@
 			)
 		)
-		(property "Description" "Resistor"
+		(property "Description" "Resistor 0 5% 0.25W SMD 0603『 』0 ohm"
 			(at 256.54 64.77 0)
 			(effects
@@
 			)
 		)
-		(property "Description" "Resistor"
+		(property "Description" "Resistor 5.1k 5% 0.25W SMD 0603『 』5.1k"
 			(at 68.58 148.59 0)
 			(effects
@@
 			)
 		)
-		(property "Description" "Unpolarized capacitor"
+		(property "Description" "Capacitor ceramic 1u 16V 10% X7R 0603『 』1u"
 			(at 261.62 146.05 0)
 			(effects
@@
 			)
 		)
-		(property "Description" "Resistor"
+		(property "Description" "Resistor 10k 5% 0.25W SMD 0603『 』10k"
 			(at 208.28 161.29 0)
 			(effects
@@
 			)
 		)
-		(property "Description" "Resistor"
+		(property "Description" "Resistor 0 5% 0.25W SMD 0603『 』0 ohm"
 			(at 382.27 109.22 0)
 			(effects
@@
 			)
 		)
-		(property "Description" "Resistor"
+		(property "Description" "Resistor 470k 1% 0.25W SMD 0603『 』470k"
 			(at 49.53 219.71 0)
 			(effects
@@
 			)
 		)
-		(property "Value" "ESP32-S3-WROOM-1"
-			(at 167.894 166.878 0)
+		(property "Value" "ESP32-S3-WROOM-1U-N16R8"
+			(at 177.8 166.878 0)
 			(effects
 				(font
@@
 			)
 		)
-		(property "Description" "Resistor"
+		(property "Description" "Resistor 2.2k 5% 0.25W SMD 0603『 』2.2k"
 			(at 123.19 207.01 0)
 			(effects
@@
 			)
 		)
-		(property "Description" "Unpolarized capacitor"
+		(property "Description" "Capacitor ceramic 1u 16V 10% X7R 0603『 』1u"
 			(at 219.71 146.05 0)
 			(effects
@@
 			)
 		)
-		(property "Description" "Resistor"
+		(property "Description" "Resistor 10k 5% 0.25W SMD 0603『 』10k"
 			(at 261.62 132.08 0)
 			(effects
@@
 			)
 		)
-		(property "Description" "Resistor"
+		(property "Description" "Resistor 10k 5% 0.25W SMD 0603『 』10k"
 			(at 367.03 161.29 0)
 			(effects
@@
 			)
 		)
-		(property "Description" "Unpolarized capacitor"
+		(property "Description" "Capacitor ceramic 100n 16V 10% X7R 0603『 』100n"
 			(at 59.69 219.71 0)
 			(effects
@@
 			)
 		)
-		(property "Description" "Resistor"
+		(property "Description" "Resistor 470k 1% 0.25W SMD 0603『 』470k"
 			(at 49.53 207.01 0)
 			(effects
@@
 			)
 		)
-		(property "Description" "Resistor"
+		(property "Description" "Resistor 470k 1% 0.25W SMD 0603『 』470k"
 			(at 97.79 219.71 0)
 			(effects
@@
 			)
 		)
-		(property "Description" "Unpolarized capacitor"
+		(property "Description" "Capacitor ceramic 22u 6.3V 10% C0G 0805『 』22u"
 			(at 175.26 222.25 0)
 			(effects
@@
 			)
 		)
-		(property "Description" "Resistor"
+		(property "Description" "Resistor 470k 1% 0.25W SMD 0603『 』470k"
 			(at 73.66 219.71 0)
 			(effects
@@
 			)
 		)
-		(property "Description" "Resistor"
+		(property "Description" "Resistor 20 ohm 5% 0.25W SMD 0603『 』20 ohm"
 			(at 295.91 101.6 0)
 			(effects
@@
 			)
 		)
-		(property "Description" "Resistor"
+		(property "Description" "Resistor 470k 1% 0.25W SMD 0603『 』470k"
 			(at 73.66 207.01 0)
 			(effects
@@
 			)
 		)
-		(property "Description" "Resistor"
+		(property "Description" "Resistor 22 ohm 5% 0.25W SMD 0603『 』22 ohm"
 			(at 123.19 127 0)
 			(effects
@@
 			)
 		)
-		(property "Description" "Resistor"
+		(property "Description" "Resistor 10k 5% 0.25W SMD 0603『 』10k"
 			(at 219.71 132.08 0)
 			(effects
@@
 			)
 		)
-		(property "Description" "Resistor"
+		(property "Description" "Resistor 0 5% 0.25W SMD 0603『 』0 ohm"
 			(at 210.82 72.39 0)
 			(effects
@@
 			)
 		)
-		(property "Description" "Unpolarized capacitor"
+		(property "Description" "Capacitor ceramic 22u 6.3V 10% C0G 0805『 』22u"
 			(at 372.11 83.82 0)
 			(effects
@@
 			)
 		)
-		(property "Description" "Resistor"
+		(property "Description" "Resistor 220k 1% 0.25W SMD 0603『 』220k"
 			(at 223.52 212.09 0)
 			(effects
@@
 			)
 		)
-		(property "Description" "Resistor"
+		(property "Description" "Resistor 10k 5% 0.25W SMD 0603『 』10k"
 			(at 48.26 41.91 0)
 			(effects
@@
 			)
 		)
-		(property "Description" "Resistor"
+		(property "Description" "Resistor 20 ohm 5% 0.25W SMD 0603『 』20 ohm"
 			(at 288.29 96.52 0)
 			(effects
@@
 			)
 		)
-		(property "Description" "Unpolarized capacitor"
+		(property "Description" "Capacitor ceramic 22u 6.3V 10% C0G 0805『 』22u"
 			(at 181.61 222.25 0)
 			(effects
@@
 			)
 		)
-		(property "Description" "Resistor"
+		(property "Description" "Resistor 0 5% 0.25W SMD 0603『 』0 ohm"
 			(at 288.29 111.76 0)
 			(effects
@@
 			)
 		)
-		(property "Description" "Resistor"
+		(property "Description" "Resistor 1.5k 5% 0.25W SMD 0603『 』1.5k"
 			(at 106.68 118.11 0)
 			(effects

Commit message: Final updates
Parts:
- J1: P/N (none) -> GT-USB-7002A
- J2: P/N (none) -> B2B-PH-K-S(LF)(SN)
- J4, J5: P/N (none) -> HY-4A
- J6: now not fitted
- TP1: now fitted
